File: PCB/Kicad Project File/ZYQ15 HE.kicad_pcb (KiCad board)
At the start: 2 copper layers, 154.3 x 110.2 mm, 130 parts, among them J1 I2C OLED, U16 ESP32-S3-DevKitC

Commit message: Updated PCB Design files
Parts:
- S1, S2: value HE Switch -> Keyswitch; footprint ScottoKeebs_MX:MX_HE_PCB_1.00u -> ScottoKeebs_Hotswap:Hotswap_MX_1.00u
- S13, S14: footprint ScottoKeebs_MX:MX_HE_PCB_1.25u -> ScottoKeebs_MX:MX_HE_PCB_1.00u
- S16, S17: value Keyswitch -> HE Switch; footprint ScottoKeebs_Hotswap:Hotswap_MX_1.00u -> ScottoKeebs_MX:MX_HE_PCB_1.25u
- moved C2 153.4 mm to (232.4, 44.2), turned to -90 degrees
- moved C6 149.6 mm to (232.4, 70.8), turned to -90 degrees
- moved C22 147.7 mm to (241.9, 58.7), turned to -90 degrees
- moved C26 146.3 mm to (241.9, 77.8), turned to -90 degrees
- moved C14 138.9 mm to (232.4, 108.9), turned to -90 degrees
- moved C10 138.9 mm to (232.4, 89.9), turned to -90 degrees
- moved C30 136.4 mm to (241.9, 96.8), turned to -90 degrees
- moved R11 135.2 mm to (228.6, 57.1)
- moved R12 135.2 mm to (228.6, 61.0)
- moved R13 135.2 mm to (228.6, 64.8)
- moved C17 134.8 mm to (227.7, 128.0), turned to -90 degrees
- moved C33 133.0 mm to (238.1, 115.9), turned to -90 degrees
- moved C5 130.3 mm to (213.4, 70.8), turned to -90 degrees
- moved R25 129.3 mm to (228.6, 83.8)
- moved R24 129.3 mm to (228.6, 80.0)
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Routing:
- net 5V: track 0.00 -> 737.0 mm, vias 0 -> 1
- net GND: track 0.00 -> 229.3 mm, vias 0 -> 1
- net 3.3V: track 0.00 -> 133.8 mm
- net Net-(D1-DIN): track 0.00 -> 98.6 mm
- net Net-(D1-DOUT): track 0.00 -> 52.4 mm
- net Net-(D16-DOUT): track 0.00 -> 19.0 mm
- net Net-(D15-DOUT): track 0.00 -> 19.0 mm
- net Net-(D8-DOUT): track 0.00 -> 14.3 mm
- net Net-(D5-DOUT): track 0.00 -> 14.3 mm
- net Net-(D4-DOUT): track 0.00 -> 14.3 mm
- net Net-(D13-DOUT): track 0.00 -> 14.3 mm
- net Net-(D12-DOUT): track 0.00 -> 14.3 mm
- net Net-(D10-DIN): track 0.00 -> 14.3 mm
- net Net-(D7-DOUT): track 0.00 -> 14.3 mm
- net Net-(D3-DOUT): track 0.00 -> 14.3 mm
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Other:
- board size 154.3 x 110.2 mm -> 118.1 x 110.5 mm

Commit message: Updated PCB design files
Parts:
- C18: footprint Capacitor_THT:CP_Radial_D10.0mm_P5.00mm -> Capacitor_THT:CP_Radial_D10.0mm_P5.00mm_BACK
- R1: value 220Ω -> 100Ω
Connections:
- U16 pad 10: 15 -> 10
- U16 pad 11: unconnected-(U16-GPIO18/ADC2_CH7-Pad11) -> 9
- U16 pad 13: 3 -> 7
- U16 pad 15: 9 -> 6
- U16 pad 16: 10 -> 5
- U16 pad 17: 11 -> 4
- U16 pad 18: 12 -> 3
- U16 pad 19: 13 -> 2
- U16 pad 20: 14 -> 1
- U16 pad 25: unconnected-(U16-GPIO19/USB_D--Pad25) -> SDA
- U16 pad 26: unconnected-(U16-GPIO20/USB_D+-Pad26) -> SCL
- U16 pad 27: SCL -> ST1
- U16 pad 28: SDA -> ST2
- U16 pad 29: DIN (LED) -> unconnected-(U16-GPIO48-Pad29)
- U16 pad 34: ST1 -> unconnected-(U16-GPIO37-Pad34)
- U16 pad 35: ST2 -> unconnected-(U16-GPIO38-Pad35)
- U16 pad 4: 4 -> unconnected-(U16-GPIO4/ADC1_CH3-Pad4)
- U16 pad 40: 2 -> unconnected-(U16-GPIO2/ADC1_CH1-Pad40)
- U16 pad 41: 1 -> unconnected-(U16-GPIO1/ADC1_CH0-Pad41)
- U16 pad 43: unconnected-(U16-GPIO43/U0TXD-Pad43) -> DIN (LED)
- U16 pad 5: 5 -> 15
- U16 pad 6: 6 -> 14
- U16 pad 7: 7 -> 13
- U16 pad 8: unconnected-(U16-GPIO15/ADC2_CH4/32K_P-Pad8) -> 12
- U16 pad 9: unconnected-(U16-GPIO16/ADC2_CH5/32K_N-Pad9) -> 11
Routing:
- net GND: track 229.3 -> 69.8 mm, vias 1 -> 9
- net ST2: track 0.00 -> 131.1 mm, vias 0 -> 1
- net ST1: track 0.00 -> 112.5 mm, vias 0 -> 1
- net Net-(D14-DOUT): track 0.00 -> 105.7 mm
- net Net-(D2-DOUT): track 0.00 -> 102.6 mm
- net Net-(D10-DOUT): track 0.00 -> 100.9 mm
- net Net-(D6-DOUT): track 0.00 -> 100.9 mm
- net SCL: track 0.00 -> 91.8 mm
- net SDA: track 0.00 -> 87.4 mm
- net 4: track 3.81 -> 84.7 mm, vias 0 -> 1
- net 8: track 3.81 -> 80.1 mm, vias 0 -> 1
- net 12: track 3.81 -> 76.4 mm, vias 0 -> 1
- net 15: track 3.81 -> 74.5 mm, vias 0 -> 1
- net 3: track 3.81 -> 63.9 mm, vias 0 -> 1
- net 7: track 3.81 -> 60.0 mm, vias 0 -> 1
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- added copper zone on B.Cu, net GND
- added copper zone on F.Cu, net GND
